File: XLD/Q1_2023/Q1_2023.kicad_sch (KiCad schematic)
At the start: 8 parts

Commit message: qw5q_gold up to date
Parts:
- added LO1: LO_R&S, symbol Quantum Computing:LO_R&S
Connections:
- new net L3-28: LO1.
Other:
- sheet QW5Q_gold QBlox ports: added none; removed 4_mod6_o1, 4_mod6_o2
- note added: "192.168.0.38"

Commit message: QM added but not labelled yet
Parts:
- renumbered L:101 to L:?, L:102 to L:?, LO1 to LO?, QPU104 to QPU?, QPU101 to QPU?, QPU103 to QPU?, QPU102 to QPU?, QPU105 to QPU?
Other:
- sheet QM_25q ports: added QM_1_I1_Q2, QM_1_I3_Q4, QM_1_I5_Q6, QM_1_I7_Q8, QM_1_I9_Q8_OUT, QM_1_IN, QM_2_5, QM_2_6, QM_2_7, QM_2_8, QM_2_I3_Q4, QM_2_I5_Q6, QM_3_1, QM_3_2, QM_4_I1_Q2, QM_4_I3_Q4, QM_4_I5_Q6, QM_4_I7_Q8, QM_4_I9_Q8_OUT, QM_4_IN, QM_5_3, QM_5_4, QM_5_5, QM_5_6, QM_5_7, QM_5_I5_Q6, QM_6_I1_Q2, QM_6_I3_Q4, QM_6_I5_Q6, QM_6_I7_Q8, QM_6_I9_Q8_OUT, QM_6_IN, QM_7_3, QM_7_4, QM_7_5, QM_7_6, QM_7_7, QM_7_I5_Q6, QM_8_7, QM_8_8, QM_9_1, QM_9_2, QM_9_3, QM_9_4, QM_9_5, QM_9_6, QM_9_7; removed none
- note added: "192.168.0.39"
- note removed: "192.168.0.38"
- moved on the sheet: LO?
