File: XLD/Q1_2023/qblox_192_168_0_20.kicad_sch (KiCad schematic)
At the start: 12 parts

Commit message: qw5q_gold up to date
Connections:
- net at IP602. (9): now also QCM_RF604. (o2); no longer QRM_RF601. (o4)
- net at QRM_RF601. (o1): now also SC601.; no longer SC602.
- net at QCM602. (o4): now also IP602. (9)
- new net: IP602. (9), QRM_RF601. (o4) (x2)
- new net: QRM_RF601. (o1), SC602.
- new net: IP602. (9), QRM_RF601. (o1) (x2)
- new net: IP602. (9), QCM_RF604. (o2)
- new net: IP602. (9), QCM_RF603. (o2)
- new net: IP602. (9), QCM601. (Trig)
- new net: QRM_RF601. (o1), SC601.

Commit message: QM added but not labelled yet
Connections:
- net at IP602. (9): now also QCM_RF604. (o2); no longer QRM_RF601. (o4)
- net at QRM_RF601. (o1): now also SC601.; no longer SC602.
- net at QCM602. (o4): now also IP602. (9)
- new net: IP602. (9), QRM_RF601. (o4) (x2)
- new net: QRM_RF601. (o1), SC602.
- new net: IP602. (9), QRM_RF601. (o1) (x2)
- new net: IP602. (9), QCM_RF604. (o2)
- new net: IP602. (9), QCM_RF603. (o2)
- new net: IP602. (9), QCM601. (Trig)
- new net: QRM_RF601. (o1), SC601.
Changed lines of the file:
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@@
         )
         (path "/9924af8b-9fcb-4325-a1dc-18dd2c4184d7/01ac70ae-656e-4c1c-b9e0-89039088ad17"
-          (reference "QRM_RF806") (unit 1)
+          (reference "QCM?") (unit 1)
         )
       )
@@
         )
         (path "/9924af8b-9fcb-4325-a1dc-18dd2c4184d7/01ac70ae-656e-4c1c-b9e0-89039088ad17"
-          (reference "QRM_RF804") (unit 1)
+          (reference "QRM_RF?") (unit 1)
         )
       )
@@
         )
         (path "/9924af8b-9fcb-4325-a1dc-18dd2c4184d7/01ac70ae-656e-4c1c-b9e0-89039088ad17"
-          (reference "QRM_RF805") (unit 1)
+          (reference "QCM?") (unit 1)
         )
       )
@@
         )
         (path "/9924af8b-9fcb-4325-a1dc-18dd2c4184d7/01ac70ae-656e-4c1c-b9e0-89039088ad17"
-          (reference "QRM801") (unit 1)
+          (reference "QRM?") (unit 1)
         )
       )
@@
         )
         (path "/9924af8b-9fcb-4325-a1dc-18dd2c4184d7/01ac70ae-656e-4c1c-b9e0-89039088ad17"
-          (reference "QCM_RF802") (unit 1)
+          (reference "QCM_RF?") (unit 1)
         )
       )
@@
         )
         (path "/9924af8b-9fcb-4325-a1dc-18dd2c4184d7/01ac70ae-656e-4c1c-b9e0-89039088ad17"
-          (reference "QCM_RF803") (unit 1)
+          (reference "QCM_RF?") (unit 1)
         )
       )
@@
         )
         (path "/9924af8b-9fcb-4325-a1dc-18dd2c4184d7/01ac70ae-656e-4c1c-b9e0-89039088ad17"
-          (reference "QCM801") (unit 1)
+          (reference "QCM?") (unit 1)
         )
       )
@@
         )
         (path "/9924af8b-9fcb-4325-a1dc-18dd2c4184d7/01ac70ae-656e-4c1c-b9e0-89039088ad17"
-          (reference "QRM_RF803") (unit 1)
+          (reference "QRM_RF?") (unit 1)
         )
       )
@@
         )
         (path "/9924af8b-9fcb-4325-a1dc-18dd2c4184d7/01ac70ae-656e-4c1c-b9e0-89039088ad17"
-          (reference "QCM_RF801") (unit 1)
-        )
-      )
+          (reference "QCM_RF?") (unit 1)
+        )
+      )
