File: XLD/Q1_2023/qm_192.168.0.1.kicad_sch (KiCad schematic)
At the start: 23 parts

Commit message: QM added but not labelled yet
Parts:
- removed LO701, LO702, LO703: LO_R&S, symbol Quantum Computing:LO_R&S
- removed OPX703, OPX704, OPX705, OPX706, OPX707: QM_OPX, symbol Quantum Computing:QM_OPX
- removed Splitter701, Splitter702, Splitter703: ZFRSC_183_S+, symbol Quantum Computing:ZFRSC_183_S+
- added BT? (x14): Bias Tee, symbol Quantum Computing:Bias Tee
- added LO1, LO2, LO3, LO4, LO5, LO6, LO7, LO8: LO_ERA_pp, symbol Quantum Computing:LO_ERA_pp
- added LO10, LO12, LO13, LO14, LO15, LO16, LO9: LO_R&S, symbol Quantum Computing:LO_R&S
- added MX? (x18): Marki_IQ, symbol Quantum Computing:Marki_IQ
- added MX? (x11): SpinQ_IQ, symbol Quantum Computing:SpinQ_IQ
- added OPX? (x7): QM_OPX, symbol Quantum Computing:QM_OPX
- added Splitter1, Splitter10, Splitter11, Splitter12, Splitter13, Splitter14, Splitter15, Splitter16, Splitter17, Splitter18, Splitter19, Splitter2, Splitter20, Splitter21, Splitter3, Splitter4, Splitter5, Splitter6, Splitter7, Splitter8, Splitter9: ZFRSC_183_S+, symbol Quantum Computing:ZFRSC_183_S+
- added Splitter22: ZFSC-2-10G+, symbol Quantum Computing:ZFSC-2-10G+
- added Ω? (x14): 50_cap, symbol Quantum Computing:50_cap
- MX?: renamed from MX706; value Mixer_IQ -> SpinQ_IQ; symbol Quantum Computing:Mixer_IQ -> Quantum Computing:SpinQ_IQ
- MX?: renamed from MX705; value Mixer_IQ -> Marki_IQ; symbol Quantum Computing:Mixer_IQ -> Quantum Computing:Marki_IQ
- MX?: renamed from MX704; value Mixer_IQ -> Marki_IQ; symbol Quantum Computing:Mixer_IQ -> Quantum Computing:Marki_IQ
- MX?: renamed from MX701; value Mixer_IQ -> SpinQ_IQ; symbol Quantum Computing:Mixer_IQ -> Quantum Computing:SpinQ_IQ
- MX?: renamed from MX703; value Mixer_IQ -> SpinQ_IQ; symbol Quantum Computing:Mixer_IQ -> Quantum Computing:SpinQ_IQ
- MX?: renamed from MX702; value Mixer_IQ -> SpinQ_IQ; symbol Quantum Computing:Mixer_IQ -> Quantum Computing:SpinQ_IQ
- renumbered BT701 to BT?, BT702 to BT?, OPX701 to OPX?, OPX702 to OPX?, Ω702701701701 to Ω?, Ω701701701701 to Ω?
Connections:
- net LO_1_split_3b is gone; now on net QM_1_IN: BT?., BT?., MX?. (RF), OPX?. (LAN), Ω?., Ω?.
- net QM_1_IN: now reaches OPX?. (LAN)
- net QM_2_IN: now reaches OPX?. (LAN)
- net QM_2_IN: now also BT?., BT?., MX?. (RF), Ω?., Ω?.
- net Drive_4GHz_3 renamed QM_1_I1_Q2
- net Drive_4GHz_4 renamed QM_1_I7_Q8
- net Drive_6GHz_1 renamed QM_1_I5_Q6
- net Drive_6GHz_2 renamed QM_1_I3_Q4
- net LO_1_split_3a renamed QM_1_I9_Q8_OUT
- new net: Splitter12., Splitter13.
- new net: Splitter11., Splitter13.
- new net: Splitter13., Splitter14.
- new net: Splitter1., Splitter3.
- new net: Splitter1., Splitter2.
- new net: Splitter16., Splitter17.
- new net: Splitter15., Splitter16.
- new net: Splitter3., Splitter6.
- new net: Splitter3., Splitter4.
- new net: Splitter10., Splitter9.
- new net: Splitter2., Splitter7.
- new net: Splitter11., Splitter9.
- new net: Splitter8., Splitter9.
- new net: Splitter2., Splitter5.
- new net: Splitter18., Splitter19.
- new net: Splitter19., Splitter20.
- new net: Splitter20., Splitter22.
- new net ERA_01: LO1., MX?. (RF)
- new net ERA_02: LO2.
- new net ERA_03: LO3., MX?. (RF)
- new net ERA_04: LO4., MX?. (RF)
- new net ERA_05: MX?. (RF)
- new net ERA_06: MX?. (RF)
- new net ERA_07: MX?. (RF)
- new net ERA_08: MX?. (RF)
- new net LO_01: LO12., MX?. (RF), MX?. (RF), MX?. (RF), MX?. (RF), MX?. (RF), Splitter19.
- new net LO_02: LO13.
- new net LO_03: LO9., MX?. (RF), MX?. (RF), MX?. (RF), MX?. (RF), MX?. (RF), MX?. (RF), MX?. (RF), MX?. (RF), Splitter1.
- new net LO_04: LO14., MX?. (RF), MX?. (RF), MX?. (RF), MX?. (RF), MX?. (RF), MX?. (RF), MX?. (RF), MX?. (RF), Splitter11.
- new net LO_05: LO10., MX?. (RF)
- new net LO_06: LO15., MX?. (RF), MX?. (RF), MX?. (RF), Splitter16.
- new net QM_2_10: MX?. (RF), OPX?. (LAN)
- new net QM_2_5: MX?. (RF), OPX?. (LAN)
- new net QM_2_7: OPX?. (LAN)
- new net QM_2_8: OPX?. (LAN)
- new net QM_2_I3_Q4: MX?. (RF), OPX?. (LAN)
- new net QM_3_1: OPX?. (LAN)
- new net QM_3_2: OPX?. (LAN)
- new net QM_4_I1_Q2: MX?. (RF), MX?. (RF), OPX?. (LAN), OPX?. (LAN)
- new net QM_4_I3_Q4: MX?. (RF), MX?. (RF), OPX?. (LAN), OPX?. (LAN)
- new net QM_4_I5_Q6: MX?. (RF), MX?. (RF), OPX?. (LAN), OPX?. (LAN)
- new net QM_4_I7_Q8: MX?. (RF), OPX?. (LAN)
- new net QM_4_I9_Q8_OUT: MX?. (RF), MX?. (RF), OPX?. (LAN), OPX?. (LAN)
- new net QM_4_IN: BT?., BT?., BT?., BT?., MX?. (RF), MX?. (RF), OPX?. (LAN), OPX?. (LAN), Ω?., Ω?., Ω?., Ω?.
- new net QM_5_10: MX?. (RF), OPX?. (LAN)
- new net QM_5_3: OPX?. (LAN)
- new net QM_5_4: OPX?. (LAN)
- new net QM_5_5: MX?. (RF), OPX?. (LAN)
- new net QM_5_7: OPX?. (LAN)
- new net QM_5_IN: BT?., BT?., MX?. (RF), OPX?. (LAN), Ω?., Ω?.
- new net QM_6_I1_Q2: MX?. (RF), OPX?. (LAN)
- new net QM_6_I3_Q4: MX?. (RF), OPX?. (LAN)
- new net QM_6_I5_Q6: MX?. (RF), OPX?. (LAN)
- new net QM_6_I7_Q8: MX?. (RF), OPX?. (LAN)
- new net QM_6_I9_Q8_OUT: MX?. (RF), OPX?. (LAN)
- new net QM_6_IN: BT?., BT?., MX?. (RF), OPX?. (LAN), Ω?., Ω?.
- new net QM_7_10: MX?. (RF), OPX?. (LAN)
- new net QM_7_3: OPX?. (LAN)
- new net QM_7_4: OPX?. (LAN)
- new net QM_7_5: MX?. (RF), OPX?. (LAN)
- new net QM_7_7: OPX?. (LAN)
- new net QM_7_IN: BT?., BT?., MX?. (RF), OPX?. (LAN), Ω?., Ω?.
- new net QM_8_7: OPX?. (LAN)
- new net QM_8_8: OPX?. (LAN)
- new net QM_9_1: OPX?. (LAN)
- new net QM_9_10: MX?. (RF), OPX?. (LAN)
- new net QM_9_2: OPX?. (LAN)
- new net QM_9_3: OPX?. (LAN)
- new net QM_9_4: OPX?. (LAN)
- new net QM_9_5: OPX?. (LAN)
- new net QM_9_6: OPX?. (LAN)
- new net QM_9_7: OPX?. (LAN)
- new net QM_9_IN: BT?., BT?., MX?. (RF), OPX?. (LAN), Ω?., Ω?.
- no-connect marks 0 -> 13
Other:
- note added: "192.168.0.31"
- note added: "192.168.0.32"
- note added: "192.168.0.33"
- note added: "192.168.0.34"
- note added: "192.168.0.35"
- note added: "192.168.0.36"
- note added: "192.168.0.39"
- note added: "192.168.000.201"
- note added: "192.168.000.202"
- note added: "192.168.000.203"
- note added: "192.168.000.204"
- note added: "192.168.000.205"
- note added: "192.168.000.206"
- note added: "192.168.000.207"
- note added: "192.168.000.208"
- note added: "Frist split to SpinQ, second split to Marki"
- moved on the sheet: BT?, MX?, OPX?, Ω?
